File: UTCape-BBHeaders.sch (KiCad schematic (older format))
At the start: 2 parts, among them J1 BBB_P8, J2 BBB_P9

Commit message: added missing title, created pdf of schematics
Other:
- note added: "BeagleBone Headers"
Changed lines of the file:
@@
 $EndComp
 $Comp
-L GND #PWR18
+L GND #PWR018
 U 1 1 54EB77B0
 P 4400 2500
-F 0 "#PWR18" H 4400 2500 30  0001 C CNN
+F 0 "#PWR018" H 4400 2500 30  0001 C CNN
 F 1 "GND" H 4400 2430 30  0001 C CNN
 F 2 "" H 4400 2500 60  0000 C CNN
@@
 $EndComp
 $Comp
-L GND #PWR22
+L GND #PWR019
 U 1 1 54EB77BF
 P 9450 5400
-F 0 "#PWR22" H 9450 5400 30  0001 C CNN
+F 0 "#PWR019" H 9450 5400 30  0001 C CNN
 F 1 "GND" H 9450 5330 30  0001 C CNN
 F 2 "" H 9450 5400 60  0000 C CNN
@@
 $EndComp
 $Comp
-L GND #PWR19
+L GND #PWR020
 U 1 1 54EB77CE
 P 9700 2500
-F 0 "#PWR19" H 9700 2500 30  0001 C CNN
+F 0 "#PWR020" H 9700 2500 30  0001 C CNN
 F 1 "GND" H 9700 2430 30  0001 C CNN
 F 2 "" H 9700 2500 60  0000 C CNN
@@
 	4000 3450 4900 3450
 $Comp
-L 3V3 #PWR21
+L 3V3 #PWR021
 U 1 1 54EBF327
 P 9900 2750
-F 0 "#PWR21" H 9900 2850 40  0001 C CNN
+F 0 "#PWR021" H 9900 2850 40  0001 C CNN
 F 1 "3V3" H 9900 2875 40  0000 C CNN
 F 2 "" H 9900 2750 60  0000 C CNN
@@
 $EndComp
 $Comp
-L 3V3 #PWR20
+L 3V3 #PWR022
 U 1 1 54EBF336
 P 7050 2750
-F 0 "#PWR20" H 7050 2850 40  0001 C CNN
+F 0 "#PWR022" H 7050 2850 40  0001 C CNN
 F 1 "3V3" H 7050 2875 40  0000 C CNN
 F 2 "" H 7050 2750 60  0000 C CNN
@@
 EndData
 $EndBitmap
+Text Notes 7350 7550 0    60   ~ 0
+BeagleBone Headers
 $EndSCHEMATC
