File: UTCape-I2C.sch (KiCad schematic (older format))
At the start: 14 parts, among them IC3 EEPROM-24LC, IC4 EEPROM-24LC

Commit message: added missing title, created pdf of schematics
Changed lines of the file:
@@
 I2C2_SDA
 $Comp
-L 3V3 #PWR7
+L 3V3 #PWR07
 U 1 1 54EC9F03
 P 3750 1450
-F 0 "#PWR7" H 3750 1550 40  0001 C CNN
+F 0 "#PWR07" H 3750 1550 40  0001 C CNN
 F 1 "3V3" H 3750 1575 40  0000 C CNN
 F 2 "" H 3750 1450 60  0000 C CNN
@@
 $EndComp
 $Comp
-L GND #PWR9
+L GND #PWR08
 U 1 1 54EC9EF4
 P 3750 2600
-F 0 "#PWR9" H 3750 2600 30  0001 C CNN
+F 0 "#PWR08" H 3750 2600 30  0001 C CNN
 F 1 "GND" H 3750 2530 30  0001 C CNN
 F 2 "" H 3750 2600 60  0000 C CNN
@@
 $EndComp
 $Comp
-L GND #PWR8
+L GND #PWR09
 U 1 1 54ECA3A4
 P 5850 2100
-F 0 "#PWR8" H 5850 2100 30  0001 C CNN
+F 0 "#PWR09" H 5850 2100 30  0001 C CNN
 F 1 "GND" H 5850 2030 30  0001 C CNN
 F 2 "" H 5850 2100 60  0000 C CNN
@@
 $EndComp
 $Comp
-L 3V3 #PWR10
+L 3V3 #PWR010
 U 1 1 54ECA48A
 P 4500 3750
-F 0 "#PWR10" H 4500 3850 40  0001 C CNN
+F 0 "#PWR010" H 4500 3850 40  0001 C CNN
 F 1 "3V3" H 4500 3875 40  0000 C CNN
 F 2 "" H 4500 3750 60  0000 C CNN
@@
 $EndComp
 $Comp
-L GND #PWR12
+L GND #PWR011
 U 1 1 54ECA49C
 P 4500 4500
-F 0 "#PWR12" H 4500 4500 30  0001 C CNN
+F 0 "#PWR011" H 4500 4500 30  0001 C CNN
 F 1 "GND" H 4500 4430 30  0001 C CNN
 F 2 "" H 4500 4500 60  0000 C CNN
@@
 $EndComp
 $Comp
-L GND #PWR11
+L GND #PWR012
 U 1 1 54ECA4AA
 P 6600 4400
-F 0 "#PWR11" H 6600 4400 30  0001 C CNN
+F 0 "#PWR012" H 6600 4400 30  0001 C CNN
 F 1 "GND" H 6600 4330 30  0001 C CNN
 F 2 "" H 6600 4400 60  0000 C CNN
@@
 $EndComp
 $Comp
-L GND #PWR13
+L GND #PWR013
 U 1 1 54ECAF2B
 P 3700 5650
-F 0 "#PWR13" H 3700 5650 30  0001 C CNN
+F 0 "#PWR013" H 3700 5650 30  0001 C CNN
 F 1 "GND" H 3700 5580 30  0001 C CNN
 F 2 "" H 3700 5650 60  0000 C CNN
@@
 $EndComp
 Wire Wire Line
-	4000 4500 4000 4600
-Wire Wire Line
-	4000 4600 4000 4950
+	4000 4500 4000 4950
 Wire Wire Line
 	5100 4600 4000 4600
@@
 Connection ~ 4500 4400
 Wire Wire Line
-	4500 4300 4500 4400
-Wire Wire Line
-	4500 4400 4500 4500
+	4500 4300 4500 4500
 Wire Wire Line
 	5100 4400 4500 4400
 Connection ~ 4500 3800
 Wire Wire Line
-	4500 3750 4500 3800
-Wire Wire Line
-	4500 3800 4500 3900
-Wire Wire Line
-	3450 3800 3700 3800
-Wire Wire Line
-	3700 3800 4000 3800
-Wire Wire Line
-	4000 3800 4500 3800
-Wire Wire Line
-	4500 3800 4900 3800
-Wire Wire Line
-	4900 3800 7000 3800
-Wire Wire Line
-	7000 3800 7250 3800
+	4500 3750 4500 3900
+Wire Wire Line
+	3450 3800 7250 3800
 Wire Wire Line
 	4900 3800 4900 4250
@@
 Connection ~ 3750 2100
 Wire Wire Line
-	3750 2000 3750 2100
-Wire Wire Line
-	3750 2100 3750 2500
-Wire Wire Line
-	3750 2500 3750 2600
+	3750 2000 3750 2600
 Wire Wire Line
 	4350 2100 3750 2100
 Connection ~ 3750 1500
 Wire Wire Line
-	3750 1450 3750 1500
-Wire Wire Line
-	3750 1500 3750 1600
-Wire Wire Line
-	3750 1500 4150 1500
-Wire Wire Line
-	4150 1500 6250 1500
-Wire Wire Line
-	6250 1500 6500 1500
+	3750 1450 3750 1600
+Wire Wire Line
+	3750 1500 6500 1500
 Wire Wire Line
 	4150 1950 4150 1500
@@
 	5100 4700 3700 4700
 Wire Wire Line
-	3700 4500 3700 4700
-Wire Wire Line
-	3700 4700 3700 4950
-Wire Wire Line
-	6300 4700 7000 4700
-Wire Wire Line
-	7000 4700 7650 4700
+	3700 4500 3700 4950
+Wire Wire Line
+	6300 4700 7650 4700
 Wire Wire Line
 	7000 4700 7000 4600
 Wire Wire Line
-	6300 4800 7250 4800
-Wire Wire Line
-	7250 4800 7650 4800
+	6300 4800 7650 4800
 Wire Wire Line
 	7250 4800 7250 4600
 Wire Wire Line
-	5550 2400 6250 2400
-Wire Wire Line
-	6250 2400 7300 2400
-Wire Wire Line
-	7300 2400 7650 2400
+	5550 2400 7650 2400
 Wire Wire Line
 	6250 2400 6250 2300
 Wire Wire Line
-	5550 2500 6500 2500
-Wire Wire Line
-	6500 2500 7000 2500
-Wire Wire Line
-	7000 2500 7650 2500
+	5550 2500 7650 2500
 Wire Wire Line
 	6500 2500 6500 2300
@@
 Connection ~ 7000 3800
 Wire Wire Line
-	3750 2500 4150 2500
-Wire Wire Line
-	4150 2500 4350 2500
-Wire Wire Line
-	4150 2300 4150 2400
-Wire Wire Line
-	4150 2400 4150 2500
+	3750 2500 4350 2500
+Wire Wire Line
+	4150 2300 4150 2500
 Wire Wire Line
 	4150 2300 4350 2300
@@
 Connection ~ 4000 4600
 Wire Wire Line
-	3700 5450 3700 5550
-Wire Wire Line
-	3700 5550 3700 5650
+	3700 5450 3700 5650
 Wire Wire Line
 	3700 5550 4000 5550
