File: UTCape-SPI.sch (KiCad schematic (older format))
At the start: 6 parts, among them IC2 EEPROM-25LC-SOT23

Commit message: added missing title, created pdf of schematics
Changed lines of the file:
@@
 $EndComp
 $Comp
-L 3V3 #PWR5
+L 3V3 #PWR05
 U 1 1 54EC6F03
 P 3600 2900
-F 0 "#PWR5" H 3600 3000 40  0001 C CNN
+F 0 "#PWR05" H 3600 3000 40  0001 C CNN
 F 1 "3V3" H 3600 3025 40  0000 C CNN
 F 2 "" H 3600 2900 60  0000 C CNN
@@
 $EndComp
 $Comp
-L GND #PWR6
+L GND #PWR06
 U 1 1 54EC6F12
 P 3600 4050
-F 0 "#PWR6" H 3600 4050 30  0001 C CNN
+F 0 "#PWR06" H 3600 4050 30  0001 C CNN
 F 1 "GND" H 3600 3980 30  0001 C CNN
 F 2 "" H 3600 4050 60  0000 C CNN
@@
 	4100 3850 3600 3850
 Wire Wire Line
-	3600 3650 3600 3850
-Wire Wire Line
-	3600 3850 3600 4050
+	3600 3650 3600 4050
 Connection ~ 3600 3850
 Wire Wire Line
@@
 	4100 3050 3600 3050
 Wire Wire Line
-	3600 2900 3600 3050
-Wire Wire Line
-	3600 3050 3600 3250
+	3600 2900 3600 3250
 Connection ~ 3600 3050
 Wire Wire Line
-	7650 3300 7050 3300
+	5650 3300 7650 3300
 Wire Wire Line
-	7050 3300 5650 3300
+	5650 3400 7650 3400
 Wire Wire Line
-	5650 3400 6750 3400
+	5650 3500 7650 3500
 Wire Wire Line
-	6750 3400 7650 3400
-Wire Wire Line
-	7650 3500 6450 3500
-Wire Wire Line
-	6450 3500 5650 3500
-Wire Wire Line
-	5650 3600 6150 3600
-Wire Wire Line
-	6150 3600 7650 3600
+	5650 3600 7650 3600
 Wire Wire Line
 	7050 3100 7050 3300
