File: UTCape-eQEP.sch (KiCad schematic (older format))
At the start: 2 parts

Commit message: added missing title, created pdf of schematics
Changed lines of the file:
@@
 GPIO3_17
 Wire Wire Line
-	4600 3450 5650 3450
+	4600 3450 6800 3450
 Wire Wire Line
-	5650 3450 6800 3450
-Wire Wire Line
-	4600 4500 5650 4500
-Wire Wire Line
-	5650 4500 6800 4500
+	4600 4500 6800 4500
 $Comp
 L TEST_POINT TP15
