File: UTCape-KiCad/UTCape.kicad_pcb (KiCad board)
At the start: 2 copper layers, 0 parts

Commit message: layed out PCB, some minor wiring changes for layout
Parts:
- added BBBCapeGuide: VAL**, BBBCapeGuide, F.Cu at (167.4, 160.3)
- added C1: 1uF, SM0603, F.Cu at (188.5, 152.1)
- added C2: 100nF, SM0603, F.Cu at (223.3, 127.3)
- added C3: 100nF, SM0603, F.Cu at (190.8, 142.6)
- added C4: 100nF, SM0603, F.Cu at (172.7, 153.4)
- added C5: 100nF, SM0603, F.Cu at (226.8, 144.9)
- added C6: 100nF, SM0603, F.Cu at (199.9, 129.3)
- added C7: 1nF, SM0603, F.Cu at (206.2, 126.5)
- added C8: 100nF, SM0603, F.Cu at (194.3, 119.6)
- added C9: 100nF, SM0603, F.Cu at (239.3, 150.6)
- added D1: 1n4148, SOD-523, F.Cu at (197.9, 119.6)
- added G***: LOGO, OSHWLOGO0.3IN, F.Cu at (244.6, 119.6)
- added IC1: 74LVC1G157, SOT363, F.Cu at (205.7, 114.6)
- added IC2: EEPROM-25LC-SOT23, SOT23_6, F.Cu at (227.1, 127.5)
- added IC3: EEPROM-24LC, SO8E, F.Cu at (194.1, 138.4)
- added IC4: EEPROM-24LC, SO8E, F.Cu at (174.5, 148.8)
- added IC5: LM555, SO8E, F.Cu at (199.9, 125.0)
- added J1: BBB_P8, H2.54-2X23, F.Cu at (215.0, 108.8)
- added J2: BBB_P9, H2.54-2X23, F.Cu at (215.0, 157.1)
- added R1: 5.6k, SM0603, F.Cu at (199.6, 137.7)
- added R10: 5.6k, SM0603, F.Cu at (226.8, 147.8)
- added R11: 10k, SM0603, F.Cu at (193.5, 127.8)
- added R12: 100, SM0603, F.Cu at (206.2, 122.9)
- added R13: 10k, SM0603, F.Cu at (193.5, 124.5)
- added R14: 10k, SM0603, F.Cu at (232.9, 150.6)
- added R2: 5.6k, SM0603, F.Cu at (197.6, 150.9)
- added R3: 5.6k, SM0603, F.Cu at (180.1, 148.8)
- added R4: 5.6k, SM0603, F.Cu at (179.6, 153.4)
- added R5: 5.6k, SM0603, F.Cu at (169.2, 143.8)
- added R6: 5.6k, SM0603, F.Cu at (172.2, 143.8)
- added R7: 5.6k, SM0603, F.Cu at (176.0, 144.0)
- added R8: 5.6k, SM0603, F.Cu at (176.0, 153.4)
- added R9: 10k, SM0603, F.Cu at (226.8, 150.6)
- added TP1: TEST_POINT, TP-5016, F.Cu at (191.0, 147.1)
- added TP10: TEST_POINT, TP-5016, F.Cu at (198.4, 146.1)
- added TP11: TEST_POINT, TP-5016, F.Cu at (205.0, 138.4)
- added TP12: TEST_POINT, TP-5016, F.Cu at (210.6, 124.0)
- added TP13: TEST_POINT, TP-5016, F.Cu at (236.0, 145.0)
- added TP14: TEST_POINT, TP-5016, F.Cu at (242.2, 145.0)
- added TP15: TEST_POINT, TP-5016, F.Cu at (247.3, 130.9)
- added TP16: TEST_POINT, TP-5016, F.Cu at (247.3, 125.0)
- added TP17: TEST_POINT, TP-5016, F.Cu at (181.6, 115.8)
- added TP2: TEST_POINT, TP-5016, F.Cu at (184.9, 147.1)
- added TP3: TEST_POINT, TP-5016, F.Cu at (214.6, 115.6)
- added TP4: TEST_POINT, TP-5016, F.Cu at (210.6, 148.3)
- added TP5: TEST_POINT, TP-5016, F.Cu at (216.7, 148.1)
- added TP6: TEST_POINT, TP-5016, F.Cu at (234.2, 132.3)
- added TP7: TEST_POINT, TP-5016, F.Cu at (234.2, 124.7)
- added TP8: TEST_POINT, TP-5016, F.Cu at (222.2, 132.8)
- added TP9: TEST_POINT, TP-5016, F.Cu at (227.1, 120.7)
Routing:
- net 3V3: track 0.00 -> 151.9 mm, vias 0 -> 3
- net GND: track 0.00 -> 109.7 mm, vias 0 -> 34
- net /BeagleBone Headers/PWM1A: track 0.00 -> 81.9 mm, vias 0 -> 3
- net /BeagleBone Headers/GPIO1_28: track 0.00 -> 72.3 mm
- net /SPI Wiring/SPI0_MISO: track 0.00 -> 69.8 mm, vias 0 -> 1
- net /BeagleBone Headers/GPIO3_17: track 0.00 -> 64.8 mm, vias 0 -> 1
- net /I2C Wiring/I2C2_SCL: track 0.00 -> 58.2 mm, vias 0 -> 1
- net /BeagleBone Headers/I2C2_SCL: track 0.00 -> 49.8 mm, vias 0 -> 1
- net /SPI Wiring/SPI0_CS0: track 0.00 -> 47.8 mm
- net /SPI Wiring/SPI0_MOSI: track 0.00 -> 35.4 mm
- net /SPI Wiring/SPI0_SCLK: track 0.00 -> 34.9 mm, vias 0 -> 1
- net /BeagleBone Headers/I2C1_SCL: track 0.00 -> 30.5 mm
- net /BeagleBone Headers/I2C1_SDA: track 0.00 -> 22.3 mm
- net /BeagleBone Headers/AIN0: track 0.00 -> 20.2 mm
- net /BeagleBone Headers/GPIO0_26: track 0.00 -> 16.7 mm
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- added copper zone on B.Cu, net GND
- added copper zone on F.Cu, net GND
Other:
- board outline added: 86.4 x 54.6 mm
- net class Default: clearance 0.254 -> 0.1524
- rule trace_clearance: 0.254 -> 0.1524
- rule via_min_drill: 0.508 -> 0.3302
- rule via_min_size: 0.889 -> 0.6858
- board text added: "1"
- board text added: "3V3"
- board text added: "555 out"
- board text added: "GND"
- board text added: "GPIO1_14/ GPIO2_1"
- board text added: "I2C1 SCL"
- board text added: "I2C1 SDA"
- board text added: "PWM1A"
- board text added: "PWM1A LPF"
- board text added: "SPI0 CS0"
- board text added: "SPI0 MISO"
- board text added: "SPI0 MOSI"
- board text added: "SPI0 SCLK"
- board text added: "U1TX-U2RX"
- board text added: "U2TX-U1RX"
- board text added: "UTCape"
- board text added: "UTCape r1"
- board text added: "eQEEP0A"
- board text added: "eQEEP0B"
- board text added: "github.com/graycatlabs/UTCape"
