File: UTCape-KiCad/UTCape-BBHeaders.sch (KiCad schematic (older format))
At the start: 2 parts, among them J1 BBB_P8, J2 BBB_P9

Commit message: added missing resistor in divider plus some protection resistors, regenerated fab files
Connections:
- net GPIO0_20: now reaches J2.41 (CLKOUT2)
- net GPIO1_28: no longer names the net of J2.12 (GPIO1_28)
Changed lines of the file:
@@
 Sheet 8 9
 Title ""
-Date "24 feb 2015"
+Date "24 mar 2015"
 Rev ""
 Comp ""
@@
 Text HLabel 6750 4650 0    60   Input ~ 0
 AIN0
-Text HLabel 10150 3250 2    60   BiDi ~ 0
-GPIO1_28
 Text HLabel 10150 3350 2    60   Output ~ 0
 PWM1A
@@
 Text HLabel 10150 4750 2    60   Input ~ 0
 eQEP0_A
-Wire Wire Line
-	10150 3250 9300 3250
 Wire Wire Line
 	9300 3350 10150 3350
@@
 03 43 83 61 8C 09 03 03 03 03 43 83 61 8C 09 03 03 03 03 43 83 61 8C 09 03 03 03 03 43 83 61 03
 60 D2 64 32 30 30 30 30 34 84 CF 1C 00 A9 00 9C 01 A8 8B 59 19 06 06 06 06 06 E9 E3 33 80 C5 FF
-07 47 25 A5 D2 E9 03 52 D8 00 00 00 00 49 45 4E 44 AE 42 60 82 4A $EndBitmap
+07 47 25 A5 D2 E9 03 52 D8 00 00 00 00 49 45 4E 44 AE 42 60 82 CF $EndBitmap
 EndData
 $EndBitmap
 Text Notes 7350 7550 0    60   ~ 0
 BeagleBone Headers
+Text HLabel 6750 4750 0    60   BiDi ~ 0
+GPIO0_20
+Wire Wire Line
+	6750 4750 7550 4750
 $EndSCHEMATC
